File: pcb/pcb.kicad_pcb (KiCad board)
At the start: 2 copper layers, 5 parts, among them J1 Conn_01x05_Pin, J2 Conn_01x16_Pin, J3 Conn_01x05_Pin

Commit message: pcb with button
Parts:
- removed J1, J3: Conn_01x05_Pin, Connector_PinHeader_2.54mm:PinHeader_1x05_P2.54mm_Vertical
- added SW1: SW_Push, Button_Switch_THT:SW_PUSH_6mm, F.Cu at (165.8, 90.8)
- added SW10: SW_Push, Button_Switch_THT:SW_PUSH_6mm, F.Cu at (176.3, 125.0)
- added SW11: SW_Push, Button_Switch_THT:SW_PUSH_6mm, F.Cu at (186.9, 90.8)
- added SW12: SW_Push, Button_Switch_THT:SW_PUSH_6mm, F.Cu at (186.9, 99.3)
- added SW13: SW_Push, Button_Switch_THT:SW_PUSH_6mm, F.Cu at (186.9, 107.9)
- added SW14: SW_Push, Button_Switch_THT:SW_PUSH_6mm, F.Cu at (186.9, 116.5)
- added SW15: SW_Push, Button_Switch_THT:SW_PUSH_6mm, F.Cu at (186.9, 125.0)
- added SW16: SW_Push, Button_Switch_THT:SW_PUSH_6mm, F.Cu at (197.4, 90.8)
- added SW17: SW_Push, Button_Switch_THT:SW_PUSH_6mm, F.Cu at (197.4, 99.3)
- added SW18: SW_Push, Button_Switch_THT:SW_PUSH_6mm, F.Cu at (197.4, 107.9)
- added SW19: SW_Push, Button_Switch_THT:SW_PUSH_6mm, F.Cu at (197.4, 116.5)
- added SW2: SW_Push, Button_Switch_THT:SW_PUSH_6mm, F.Cu at (165.8, 99.3)
- added SW20: SW_Push, Button_Switch_THT:SW_PUSH_6mm, F.Cu at (197.4, 125.0)
- added SW21: SW_Push, Button_Switch_THT:SW_PUSH_6mm, F.Cu at (208.0, 90.8)
- added SW22: SW_Push, Button_Switch_THT:SW_PUSH_6mm, F.Cu at (208.0, 99.3)
- added SW23: SW_Push, Button_Switch_THT:SW_PUSH_6mm, F.Cu at (208.0, 107.9)
- added SW24: SW_Push, Button_Switch_THT:SW_PUSH_6mm, F.Cu at (208.0, 116.5)
- added SW25: SW_Push, Button_Switch_THT:SW_PUSH_6mm, F.Cu at (208.0, 125.0)
- added SW3: SW_Push, Button_Switch_THT:SW_PUSH_6mm, F.Cu at (165.8, 107.9)
- added SW4: SW_Push, Button_Switch_THT:SW_PUSH_6mm, F.Cu at (165.8, 116.5)
- added SW5: SW_Push, Button_Switch_THT:SW_PUSH_6mm, F.Cu at (165.8, 125.0)
- added SW6: SW_Push, Button_Switch_THT:SW_PUSH_6mm, F.Cu at (176.3, 90.8)
- added SW7: SW_Push, Button_Switch_THT:SW_PUSH_6mm, F.Cu at (176.3, 99.3)
- added SW8: SW_Push, Button_Switch_THT:SW_PUSH_6mm, F.Cu at (176.3, 107.9)
- added SW9: SW_Push, Button_Switch_THT:SW_PUSH_6mm, F.Cu at (176.3, 116.5)
